Commit message: Merged PR 2897: Merge v1.6.0 into master
Related work items: #18239, #26469, #26914, #27030, #27687, #27790, #27859

File: src/assets/robots/igus/delta/delta.xacro (robot description, xacro)
@@ -10,8 +10,8 @@
             <origin rpy="0 0 0" xyz="0 0 0"/>
             <geometry>
-                <mesh filename="./meshes/visual/body4.stl"/>
+                <mesh filename="./meshes/visual/body.dae"/>
             </geometry>
             <material name="">
-                <color rgba="0 0 0 0.2"/>
+                <color rgba="1 0 0 0.2"/>
             </material>
         </visual>

File: src/assets/robots/midea/wukong500/wukong500.xacro (robot description, xacro)
@@ -58,6 +58,6 @@
                               origin="0.225 0 0.075" parent="link1" child="link2"/>
     <xacro:def_link link_name="link2" mesh_name="link2.dae"/>
-    <xacro:def_prismatic_joint joint_name="joint3" axis="0 0 1" effort="1000.0" lower="-0.1315" upper="0.01"
-                               velocity="1.0" origin="0.274 0 0.015" parent="link2" child="link_empty_1"/>
+    <xacro:def_prismatic_joint joint_name="joint3" axis="0 0 1" effort="1000.0" lower="-14" upper="0.1"
+                               velocity="1.0" origin="0.274 0 0.02" parent="link2" child="link_empty_1"/>
     <xacro:def_empty_link link_name="link_empty_1"/>
     <xacro:def_revolute_joint joint_name="joint4" axis="0 0 1" effort="1000.0" lower="-360" upper="360" velocity="1.0"
